File: hardware/bitsy-v0.3a/icebreaker-bitsy.kicad_pcb (KiCad board)
At the start: 4 copper layers, 38.1 x 17.8 mm, 101 parts, among them J1 Conn_01x01, J10 Conn_01x01, J11 Conn_01x01, J12 Conn_01x01, J13 Conn_01x01, J14 Jumper, J15 Jumper, J16 Jumper, J17 Jumper, J18 Jumper, J19 Jumper, J2 Conn_01x01, J20 Conn_01x01, J21 Conn_01x01, J22 Conn_01x01, J23 Conn_01x01, J24 Conn_01x01, J25 Conn_01x01, J26 Conn_01x01, J27 Conn_01x01, J28 Conn_01x01, J29 Conn_01x01, J3 Conn_01x01, J30 Conn_01x01, J31 Conn_01x01, J32 Conn_01x01, J33 Conn_01x01, J34 Conn_01x01, J35 Conn_01x01, J36 Conn_01x01, J37 Conn_01x01, J38 Jumper, J39 Jumper, J4 Conn_01x01, J40 Jumper, J41 Conn_01x01, J42 Conn_01x01, J43 Conn_01x01, J44 Conn_01x01, J45 Conn_01x01, J46 Conn_01x01, J47 Conn_01x01, J48 Conn_01x01, J49 Conn_01x01, J5 Conn_01x01, J6 Conn_01x01, J7 Conn_01x01, J8 Conn_01x01, J9 Conn_01x01, P1 USB_OTG, P2 UP, P3 UP, P4 UP, P5 UP, SW1 TACT, U1 USBLC6-2, U2 3.3V, U3 1V2, U4 LY68L6400, U5 W25Q, U6 ICE5LP4K-SG48, X1 DSC6101CI1A-012.0000T

Commit message: Minor cleanups, finishing up for prototype order.
This is the status from the ad hoc stream from Apr 4th 2020.
Parts:
- REF**: value null_Logo_SilkS_5mm -> 1b2_Logo_SilkS_6.5mm; footprint pkl_logos:null_Logo_SilkS_5mm -> pkl_logos:1b2_Logo_SilkS_6.5mm
- moved REF** 0.50 mm to (48.8, 47.5)
Routing:
- net GND: vias 19 -> 28
Other:
- board text added: "1BitSquared"
- board text added: "LEDB"
- board text added: "LEDG"
- board text added: "LEDR"
- board text added: "VCCIO01"
- board text added: "vpp2v5"
- board text removed: "NULL"
