File: hardware/bitsy-v0.3b/icebreaker-bitsy.kicad_pcb (KiCad board)
At the start: 4 copper layers, 38.1 x 17.8 mm, 101 parts, among them J1 Conn_01x01, J10 Conn_01x01, J11 Conn_01x01, J12 Conn_01x01, J13 Conn_01x01, J14 Jumper, J15 Jumper, J16 Jumper, J17 Jumper, J18 Jumper, J19 Jumper, J2 Conn_01x01, J20 Conn_01x01, J21 Conn_01x01, J22 Conn_01x01, J23 Conn_01x01, J24 Conn_01x01, J25 Conn_01x01, J26 Conn_01x01, J27 Conn_01x01, J28 Conn_01x01, J29 Conn_01x01, J3 Conn_01x01, J30 Conn_01x01, J31 Conn_01x01, J32 Conn_01x01, J33 Conn_01x01, J34 Conn_01x01, J35 Conn_01x01, J36 Conn_01x01, J37 Conn_01x01, J38 Jumper, J39 Jumper, J4 Conn_01x01, J40 Jumper, J41 Conn_01x01, J42 Conn_01x01, J43 Conn_01x01, J44 Conn_01x01, J45 Conn_01x01, J46 Conn_01x01, J47 Conn_01x01, J48 Conn_01x01, J49 Conn_01x01, J5 Conn_01x01, J6 Conn_01x01, J7 Conn_01x01, J8 Conn_01x01, J9 Conn_01x01, P1 USB_OTG, P2 UP, P3 UP, P4 UP, P5 UP, SW1 TACT, U1 USBLC6-2, U2 3.3V, U3 1V2, U4 LY68L6400, U5 W25Q, U6 ICE5LP4K-SG48, X1 DSC6101CI1A-012.0000T

Commit message: Clean up routing
Parts:
- moved C27 1.15 mm to (44.9, 52.9)
- moved C36 1.15 mm to (47.9, 52.9)
- moved C37 1.15 mm to (46.9, 52.9)
- moved C38 1.15 mm to (45.9, 52.9)
- moved R19 1.15 mm to (48.9, 52.9)
- moved J18 0.24 mm to (61.8, 42.6), turned to 0 degrees
- moved J17 0.18 mm to (44.9, 52.9)
- turned C23 to 90 degrees
Routing:
- net /ICEVCC: track 31.4 -> 12.4 mm, vias 4 -> 3
- net /~LEDG: track 24.0 -> 27.9 mm
- net +3V3: track 27.7 -> 25.3 mm
- net /FLASH_~WP~-IO2: track 32.6 -> 30.8 mm, vias 5 -> 4
- net /IOB_23B: track 20.0 -> 21.8 mm
- net /CLK: track 12.3 -> 14.1 mm
- net /~BUTTON: track 20.0 -> 18.3 mm
- net /IOB_29B: track 18.5 -> 20.2 mm
- net /IOT_37A: track 20.8 -> 19.5 mm
- net Net-(D1-Pad4): track 7.10 -> 8.43 mm
- net /FLASH_~HLD~-~RST~-IO3: track 27.2 -> 26.1 mm
- net /UVBUS: track 5.43 -> 6.38 mm
- net /IOT_44B: track 7.47 -> 8.39 mm
- net /~LED_RED: track 18.7 -> 17.9 mm
- net +5V: track 27.7 -> 28.5 mm
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Other:
- rule pad_to_mask_clearance: 0.05 -> 0.025
- board text added: "1Bit Squared 2020"
- board text removed: "1Bitsquared 2020"
